File: hardware/prototype/prototype/prototype.kicad_pcb (KiCad board)
At the start: 2 copper layers, 26.7 x 240.3 mm, 52 parts, among them J1 Conn_01x10_Male, J2 USB_C_Receptacle_USB2.0

Commit message: Update proto bar
Parts:
- removed C10, C11, C12, C13, C14, C15, C16, C17, C18, C19, C20, C21, C22, C23, C24, C25, C9: 104, Capacitor_SMD:C_0805_2012Metric
- removed D17, D18, D19, D20, D21, D22, D23, D24, D25: WS2812B, LED_SMD:LED_WS2812B_PLCC4_5.0x5.0mm_P3.2mm
- C1, C2, C3, C4, C5, C6, C7, C8: value 104 -> 0.1uF; footprint Capacitor_SMD:C_0805_2012Metric -> Capacitor_SMD:C_0603_1608Metric
- D1, D10, D11, D12, D13, D14, D15, D16, D2, D3, D4, D5, D6, D7, D8, D9: value WS2812B -> APA102; footprint LED_SMD:LED_WS2812B_PLCC4_5.0x5.0mm_P3.2mm -> LED_SMD:LED_RGB_5050-6
- J1: value Conn_01x10_Male -> BAR Debug; footprint Connector_PinHeader_2.54mm:PinHeader_1x10_P2.54mm_Horizontal -> Connector_PinHeader_2.54mm:PinHeader_1x04_P2.54mm_Horizontal
- moved J1 165.1 mm to (46.0, 59.9), turned to 90 degrees
- moved C8 96.4 mm to (40.1, 189.0), turned to 270 degrees
- moved C7 88.3 mm to (40.1, 172.0), turned to 270 degrees
- moved C6 80.4 mm to (40.1, 155.2), turned to 270 degrees
- moved C5 72.3 mm to (40.1, 138.2), turned to 270 degrees
- moved C4 63.8 mm to (40.1, 120.7), turned to 270 degrees
- moved J2 60.2 mm to (42.2, 205.0)
- moved C3 56.2 mm to (40.1, 104.2), turned to 270 degrees
- moved C2 48.4 mm to (40.1, 87.1), turned to 270 degrees
- moved C1 41.2 mm to (40.1, 70.6), turned to 270 degrees
- moved D1 34.2 mm to (43.7, 66.3), turned to 270 degrees
- moved D2 33.7 mm to (43.7, 74.7), turned to 270 degrees
- moved D3 33.2 mm to (43.7, 83.2), turned to 270 degrees
- moved D4 32.6 mm to (43.7, 91.3), turned to 270 degrees
- moved D5 32.2 mm to (43.7, 99.8), turned to 270 degrees
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Connections:
- D1 pad 1: +5V -> /LED BAR/BAR_DI
- D1 pad 2: Net-(D1-Pad2) -> /LED BAR/BAR_CI
- D1 pad 4: /LED BAR/LED_G1_DIN -> +5V
- D10 pad 1: +5V -> Net-(D10-Pad1)
- D10 pad 2: /LED BAR/LED_G2_DOUT -> Net-(D10-Pad2)
- D10 pad 4: Net-(D10-Pad4) -> +5V
- D11 pad 1: +5V -> Net-(D10-Pad6)
- D11 pad 2: Net-(D11-Pad2) -> Net-(D10-Pad5)
- D11 pad 4: /LED BAR/LED_G3_DIN -> +5V
- D12 pad 1: +5V -> Net-(D11-Pad6)
- D12 pad 2: Net-(D12-Pad2) -> Net-(D11-Pad5)
- D12 pad 4: Net-(D11-Pad2) -> +5V
- D13 pad 1: +5V -> Net-(D12-Pad6)
- D13 pad 2: Net-(D13-Pad2) -> Net-(D12-Pad5)
- D13 pad 4: Net-(D12-Pad2) -> +5V
- D14 pad 1: +5V -> Net-(D13-Pad6)
- D14 pad 2: Net-(D14-Pad2) -> Net-(D13-Pad5)
- D14 pad 4: Net-(D13-Pad2) -> +5V
- D15 pad 1: +5V -> Net-(D14-Pad6)
- D15 pad 2: /LED BAR/LED_G3_DOUT -> Net-(D14-Pad5)
- D15 pad 4: Net-(D14-Pad2) -> +5V
- D16 pad 1: +5V -> Net-(D15-Pad6)
- D16 pad 2: Net-(D16-Pad2) -> Net-(D15-Pad5)
- D16 pad 4: /LED BAR/LED_G4_DIN -> +5V
- D2 pad 1: +5V -> Net-(D1-Pad6)
- D2 pad 2: Net-(D2-Pad2) -> Net-(D1-Pad5)
- D2 pad 4: Net-(D1-Pad2) -> +5V
- D3 pad 1: +5V -> Net-(D2-Pad6)
- D3 pad 2: Net-(D3-Pad2) -> Net-(D2-Pad5)
- D3 pad 4: Net-(D2-Pad2) -> +5V
- D4 pad 1: +5V -> Net-(D3-Pad6)
- D4 pad 2: Net-(D4-Pad2) -> Net-(D3-Pad5)
- D4 pad 4: Net-(D3-Pad2) -> +5V
- D5 pad 1: +5V -> Net-(D4-Pad6)
- D5 pad 2: /LED BAR/LED_G1_DOUT -> Net-(D4-Pad5)
- D5 pad 4: Net-(D4-Pad2) -> +5V
- D6 pad 1: +5V -> Net-(D5-Pad6)
- D6 pad 2: Net-(D6-Pad2) -> Net-(D5-Pad5)
- D6 pad 4: /LED BAR/LED_G2_DIN -> +5V
- D7 pad 1: +5V -> Net-(D6-Pad6)
- D7 pad 2: Net-(D7-Pad2) -> Net-(D6-Pad5)
- D7 pad 4: Net-(D6-Pad2) -> +5V
- D8 pad 1: +5V -> Net-(D7-Pad6)
- D8 pad 2: Net-(D8-Pad2) -> Net-(D7-Pad5)
- D8 pad 4: Net-(D7-Pad2) -> +5V
- D9 pad 1: +5V -> Net-(D8-Pad6)
- D9 pad 2: Net-(D10-Pad4) -> Net-(D8-Pad5)
- D9 pad 4: Net-(D8-Pad2) -> +5V
- J1 pad 1: /LED BAR/LED_G1_DIN -> /LED BAR/BAR_DI
- J1 pad 2: /LED BAR/LED_G1_DOUT -> /LED BAR/BAR_CI
- J1 pad 3: /LED BAR/LED_G2_DIN -> /LED BAR/BAR_DO
- J1 pad 4: /LED BAR/LED_G2_DOUT -> /LED BAR/BAR_CO
- J2 pad S1: Net-(J2-PadS1) -> GND
Routing:
- net GND: track 584.1 -> 113.2 mm, vias 0 -> 16
- net +5V: track 366.3 -> 71.2 mm, vias 0 -> 16
- net /LED BAR/LED_G1_DIN: track 200.6 -> 0.00 mm
- net /LED BAR/LED_G1_DOUT: track 168.1 -> 0.00 mm
- net /LED BAR/LED_G2_DIN: track 162.8 -> 0.00 mm
- net /LED BAR/BAR_DO: track 0.00 -> 144.5 mm, vias 0 -> 1
- net /LED BAR/BAR_CO: track 0.00 -> 142.1 mm, vias 0 -> 1
- net /LED BAR/LED_G2_DOUT: track 129.0 -> 0.00 mm
- net /LED BAR/LED_G3_DIN: track 123.8 -> 0.00 mm
- net /LED BAR/LED_G3_DOUT: track 90.3 -> 0.00 mm
- net /LED BAR/LED_G4_DIN: track 84.1 -> 0.00 mm
- net /LED BAR/LED_G4_DOUT: track 52.0 -> 0.00 mm
- net /LED BAR/LED_G5_DIN: track 45.3 -> 0.00 mm
- net /LED BAR/LED_G5_DOUT: track 15.7 -> 0.00 mm
- net Net-(D16-Pad2): track 8.43 -> 0.00 mm
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- added copper zone on B.Cu, net +5V
- added copper zone on B.Cu, net GND
Other:
- board size 26.7 x 240.3 mm -> 11.2 x 153.5 mm
