File: hardware/prototype/prototype/prototype.sch (KiCad schematic (older format))
At the start: 2 parts, among them J1 Conn_01x10_Male, J2 USB_C_Receptacle_USB2.0

Commit message: Update proto bar
Parts:
- removed J1: Conn_01x10_Male, Connector_PinHeader_2.54mm:PinHeader_1x10_P2.54mm_Horizontal, symbol Connector:Conn_01x10_Male
- added J1: BAR Debug, Connector_PinHeader_2.54mm:PinHeader_1x04_P2.54mm_Horizontal, symbol Connector:Conn_01x04_Male
Connections:
- net GND: now also J2.S1 (SHIELD)
- new net LED BAR/BAR_CI: J1.2 (Pin_2)
- new net LED BAR/BAR_CO: J1.4 (Pin_4)
- new net LED BAR/BAR_DI: J1.1 (Pin_1)
- new net LED BAR/BAR_DO: J1.3 (Pin_3)
- no-connect marks 0 -> 8
Other:
- note removed: "Prototype\nLed debug pins"
- moved on the sheet: J2
Changed lines of the file:
@@
 $EndDescr
-$Comp
-L Connector:Conn_01x10_Male J1
-U 1 1 603C6518
-P 4150 1900
-F 0 "J1" H 4122 1874 50  0000 R CNN
-F 1 "Conn_01x10_Male" H 4122 1783 50  0000 R CNN
-F 2 "Connector_PinHeader_2.54mm:PinHeader_1x10_P2.54mm_Horizontal" H 4150 1900 50  0001 C CNN
-F 3 "~" H 4150 1900 50  0001 C CNN
-	1    4150 1900
-	-1   0    0    -1
-$EndComp
-Text Notes 4250 1650 0    50   ~ 0
-Prototype\nLed debug pins
-$Sheet
-S 1050 1350 850  1400
-U 6035AF6C
-F0 "LED BAR" 50
-F1 "led-bar.sch" 50
-F2 "LED_G1_DIN" I R 1900 1500 50
-F3 "LED_G1_DOUT" I R 1900 1600 50
-F4 "LED_G2_DIN" I R 1900 1700 50
-F5 "LED_G2_DOUT" I R 1900 1800 50
-F6 "LED_G3_DIN" I R 1900 1900 50
-F7 "LED_G3_DOUT" I R 1900 2000 50
-F8 "LED_G4_DIN" I R 1900 2100 50
-F9 "LED_G4_DOUT" I R 1900 2200 50
-F10 "LED_G5_DIN" I R 1900 2300 50
-F11 "LED_G5_DOUT" I R 1900 2400 50
-$EndSheet
-Wire Wire Line
-	1900 1500 3950 1500
-Wire Wire Line
-	3950 1600 1900 1600
-Wire Wire Line
-	1900 1700 3950 1700
-Wire Wire Line
-	1900 1800 3950 1800
-Wire Wire Line
-	3950 1900 1900 1900
-Wire Wire Line
-	1900 2000 3950 2000
-Wire Wire Line
-	3950 2100 1900 2100
-Wire Wire Line
-	1900 2200 3950 2200
-Wire Wire Line
-	3950 2300 1900 2300
-Wire Wire Line
-	3950 2400 1900 2400
 $Comp
 L power:GND #PWR0101
 U 1 1 6044D2CA
-P 1450 5200
-F 0 "#PWR0101" H 1450 4950 50  0001 C CNN
-F 1 "GND" H 1455 5027 50  0000 C CNN
-F 2 "" H 1450 5200 50  0001 C CNN
-F 3 "" H 1450 5200 50  0001 C CNN
-	1    1450 5200
+P 1400 4500
+F 0 "#PWR0101" H 1400 4250 50  0001 C CNN
+F 1 "GND" H 1405 4327 50  0000 C CNN
+F 2 "" H 1400 4500 50  0001 C CNN
+F 3 "" H 1400 4500 50  0001 C CNN
+	1    1400 4500
 	1    0    0    -1
 $EndComp
@@
 L power:+5V #PWR0102
 U 1 1 6044DA40
-P 2200 3200
-F 0 "#PWR0102" H 2200 3050 50  0001 C CNN
-F 1 "+5V" H 2215 3373 50  0000 C CNN
-F 2 "" H 2200 3200 50  0001 C CNN
-F 3 "" H 2200 3200 50  0001 C CNN
-	1    2200 3200
+P 2150 2450
+F 0 "#PWR0102" H 2150 2300 50  0001 C CNN
+F 1 "+5V" H 2165 2623 50  0000 C CNN
+F 2 "" H 2150 2450 50  0001 C CNN
+F 3 "" H 2150 2450 50  0001 C CNN
+	1    2150 2450
 	1    0    0    -1
 $EndComp
 Wire Wire Line
-	2050 3400 2200 3400
+	2000 2650 2150 2650
 Wire Wire Line
-	2200 3400 2200 3200
-Wire Wire Line
-	1450 5200 1450 4900
+	2150 2650 2150 2450
 $Comp
 L Connector:USB_C_Receptacle_USB2.0 J2
 U 1 1 6044F323
-P 1450 4000
-F 0 "J2" H 1557 4867 50  0000 C CNN
-F 1 "USB_C_Receptacle_USB2.0" H 1557 4776 50  0000 C CNN
-F 2 "Connector_USB:USB_C_Receptacle_HRO_TYPE-C-31-M-12" H 1600 4000 50  0001 C CNN
-F 3 "https://www.usb.org/sites/default/files/documents/usb_type-c.zip" H 1600 4000 50  0001 C CNN
-	1    1450 4000
+P 1400 3250
+F 0 "J2" H 1507 4117 50  0000 C CNN
+F 1 "USB_C_Receptacle_USB2.0" H 1507 4026 50  0000 C CNN
+F 2 "Connector_USB:USB_C_Receptacle_HRO_TYPE-C-31-M-12" H 1550 3250 50  0001 C CNN
+F 3 "https://www.usb.org/sites/default/files/documents/usb_type-c.zip" H 1550 3250 50  0001 C CNN
+	1    1400 3250
 	1    0    0    -1
 $EndComp
+$Sheet
+S 1050 1300 800  700
+U 6035AF6C
+F0 "LED BAR" 50
+F1 "led-bar.sch" 50
+F2 "BAR_DI" I R 1850 1450 50
+F3 "BAR_CI" I R 1850 1550 50
+F4 "BAR_DO" I R 1850 1650 50
+F5 "BAR_CO" I R 1850 1750 50
+$EndSheet
+$Comp
+L Connector:Conn_01x04_Male J1
+U 1 1 605779DE
+P 3850 1550
+F 0 "J1" H 3822 1524 50  0000 R CNN
+F 1 "BAR Debug" H 3822 1433 50  0000 R CNN
+F 2 "Connector_PinHeader_2.54mm:PinHeader_1x04_P2.54mm_Horizontal" H 3850 1550 50  0001 C CNN
+F 3 "~" H 3850 1550 50  0001 C CNN
+	1    3850 1550
+	-1   0    0    -1
+$EndComp
+Wire Wire Line
+	1100 4150 1100 4300
+Wire Wire Line
+	1100 4300 1400 4300
+Connection ~ 1400 4300
+Wire Wire Line
+	1400 4300 1400 4150
+NoConn ~ 2000 3850
+NoConn ~ 2000 3750
+NoConn ~ 2000 3450
+NoConn ~ 2000 3350
+NoConn ~ 2000 3250
+NoConn ~ 2000 3150
+NoConn ~ 2000 2950
+NoConn ~ 2000 2850
+Wire Wire Line
+	1850 1450 3650 1450
+Wire Wire Line
+	1850 1550 3650 1550
+Wire Wire Line
+	1850 1650 3650 1650
+Wire Wire Line
+	1850 1750 3650 1750
+$Comp
+L power:PWR_FLAG #FLG0101
+U 1 1 605D8E38
+P 2450 2450
+F 0 "#FLG0101" H 2450 2525 50  0001 C CNN
+F 1 "PWR_FLAG" H 2450 2623 50  0000 C CNN
+F 2 "" H 2450 2450 50  0001 C CNN
+F 3 "~" H 2450 2450 50  0001 C CNN
+	1    2450 2450
+	1    0    0    -1
+$EndComp
+Wire Wire Line
+	2450 2450 2450 2650
+Wire Wire Line
+	2450 2650 2150 2650
+Connection ~ 2150 2650
+Wire Wire Line
+	1400 4300 1400 4500
 $EndSCHEMATC
